File: Gen3.1_Printhead/Nozzle/Nozzle.kicad_pcb (KiCad board)
At the start: 2 copper layers, 49.6 x 102.6 mm, 74 parts, among them J1 IDC Conn

Commit message: adding in Gen3.1a Conector PCB inlet modifications - hole reduced from 1.27mm to 1mm, or 0.8mm
Parts:
- H63: renamed from H29; value M1.2 -> M1; footprint Pauls_KiCAD_Libraries:MountingHole_1.2mm -> Pauls_KiCAD_Libraries:MountingHole_1mm
- H64: renamed from H31; value M1.2 -> M1; footprint Pauls_KiCAD_Libraries:MountingHole_1.2mm -> Pauls_KiCAD_Libraries:MountingHole_1mm
- H65: renamed from H38; value M1.2 -> M0.8; footprint Pauls_KiCAD_Libraries:MountingHole_1.2mm -> Pauls_KiCAD_Libraries:MountingHole_0.8mm
- H66: renamed from H25; value M1.2 -> M1; footprint Pauls_KiCAD_Libraries:MountingHole_1.2mm -> Pauls_KiCAD_Libraries:MountingHole_1mm
- H67: renamed from H34; value M1.2 -> M1; footprint Pauls_KiCAD_Libraries:MountingHole_1.2mm -> Pauls_KiCAD_Libraries:MountingHole_1mm
- H68: renamed from H36; value M1.2 -> M0.8; footprint Pauls_KiCAD_Libraries:MountingHole_1.2mm -> Pauls_KiCAD_Libraries:MountingHole_0.8mm
- H69: renamed from H26; value M1.2 -> M1; footprint Pauls_KiCAD_Libraries:MountingHole_1.2mm -> Pauls_KiCAD_Libraries:MountingHole_1mm
- H70: renamed from H27; value M1.2 -> M1; footprint Pauls_KiCAD_Libraries:MountingHole_1.2mm -> Pauls_KiCAD_Libraries:MountingHole_1mm
- H71: renamed from H21; value M1.2 -> M1; footprint Pauls_KiCAD_Libraries:MountingHole_1.2mm -> Pauls_KiCAD_Libraries:MountingHole_1mm
- moved H71 0.09 mm to (148.4, 63.4)
- renumbered H39 to H1, H47 to H10, H48 to H11, H49 to H12, H50 to H13, H10 to H14, H51 to H15, H52 to H16, H53 to H17, H54 to H18, H55 to H19, H40 to H2, H56 to H20, H57 to H21, H58 to H22, H11 to H23, H1 to H24, H59 to H25, H60 to H26, H61 to H27, H62 to H28, H2 to H29, H41 to H3, H12 to H30, H63 to H31, H3 to H32, H4 to H33, H5 to H34, H6 to H35, H7 to H36, H13 to H37, H14 to H38, H8 to H39, H42 to H4, H64 to H40, H15 to H41, H16 to H42, H70 to H43, H17 to H44, H18 to H45, H71 to H46, H19 to H47, H20 to H48, H72 to H49, H43 to H5, H66 to H50, H67 to H51, H23 to H52, H22 to H53, H68 to H54, H24 to H55, H33 to H56, H69 to H57, H35 to H58, H28 to H59, H44 to H6, H37 to H60, H30 to H61, H32 to H62, H9 to H7, H45 to H8, H46 to H9
Other:
- board text added: "OPJ: V3.1a"
- board text removed: "OPJ: V3.1"

Commit message: updated Printhead to Gen3.1b - Nozzle screw holes swapped from 1.27mm to 0.635mm. Added labels to each board to help with identification
Parts:
- moved H1 1.54 mm to (147.6, 35.6)
- moved H15 1.54 mm to (127.3, 35.7)
- moved H2 1.54 mm to (132.4, 35.7)
- moved H40 1.54 mm to (146.5, 33.1)
- moved H43 1.54 mm to (131.3, 33.1)
- moved H46 1.54 mm to (144.0, 33.1)
- moved H49 1.54 mm to (128.7, 33.1)
- moved H50 1.54 mm to (141.4, 33.1)
- moved H51 1.54 mm to (138.9, 33.1)
- moved H57 1.54 mm to (133.8, 33.1)
- moved H8 1.54 mm to (137.5, 35.7)
- moved H9 1.54 mm to (142.6, 35.6)
- moved H16 1.54 mm to (129.9, 30.6)
- moved H21 1.54 mm to (134.9, 30.6)
- moved H22 1.54 mm to (145.1, 30.6)
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Other:
- board size 49.6 x 102.6 mm -> 49.6 x 103.6 mm
- board text added: "A"
- board text added: "B"
- board text added: "C"
- board text added: "D"
- board text added: "OPJ: V3.1b"
- board text removed: "OPJ: V3.1a"

Commit message: Repo now has an updated panel with 3mm holes in top plate.  Each layer is alphabet coded.
Other:
- board text added: "Open PyroJet PrintHead Gen3.1b"
- board text removed: "Open PyroJet PrintHead Gen3.1"
