File: Printhead-Controller/Printhead-Controller.sch (KiCad schematic (older format))
At the start: 44 parts, among them J1 Serial Prog, J2 OLED Screen, J3 2 x 10 Pinheader, Q1 AO3400A, SW1 Rotary_Encoder, SW2 USER1, SW3 BOOT, SW4 RESET, U1 ESP32-WROOM-32D

Commit message: final PCB KiCAD design files for V0.5 as sent off for manufacture at JLCPCB 2022-03-22
Parts:
- added J5: Nozzle2 Board (Future), Connector_PinHeader_2.54mm:PinHeader_1x04_P2.54mm_Vertical, symbol Connector_Generic:Conn_01x04
Connections:
- net GND: now also J5.1 (Pin_1)
- net EN_24V: now reaches U1.14 (IO12)
- net EN_24V: now also J5.3 (Pin_3)
- net EN_3.3V: now reaches U1.24 (IO2)
- net EN_3.3V: now also J5.2 (Pin_2)
- net EN_VSW: now reaches U1.9 (IO33)
- net EN_VSW: now also J5.4 (Pin_4)
- no-connect marks 13 -> 10
Other:
- note added: "1 easy to use spare RO GPIO"
- note added: "2 extra spare strapping pin GPIO"
- note added: "EN_24V"
- note added: "EN_3.3V"
- note added: "EN_VSW"
- note added: "GND"
- note removed: "1 easy to use spare GPIO"
- note removed: "4 extra spare strapping pin GPIO"
Changed lines of the file:
@@
 Sheet 1 2
 Title "Open-PyroJet"
-Date "2022-03-16"
-Rev "0.5c1"
+Date "2022-03-22"
+Rev "0.5c2"
 Comp "OPJ"
 Comment1 "PRL"
@@
 	3245 1875 3170 1875
 NoConn ~ 3170 1975
-NoConn ~ 3170 2075
 NoConn ~ 3170 2375
-NoConn ~ 3245 1675
 Text Notes 2125 3790 0    50   ~ 0
 Input Only:\nPin4 - GPIO36\nPin5 - GPIO39\nPin6 - GPIO34\nPin7 - GPIO35\nPin8 - GPIO39\n
@@
 Wire Wire Line
 	3245 3475 3170 3475
-Text Notes 1085 5650 0    50   ~ 0
+Text Notes 970  4915 0    50   ~ 0
 Design Philosophy:\n* over engineered to enable experimentation and exploration of a filament and nozzle limits\n* cost is not a big driver for this design, but it has been taken into account\n* not much thought on mounting issues, but this version will have to be mounted close to the printhead
-Text Notes 3885 3250 0    50   ~ 0
-1 easy to use spare GPIO
-Text Notes 3640 2055 0    50   ~ 0
-4 extra spare strapping pin GPIO
+Text Notes 3635 3695 0    50   ~ 0
+1 easy to use spare RO GPIO
+Text Notes 3600 1990 0    50   ~ 0
+2 extra spare strapping pin GPIO
 Wire Wire Line
 	3245 3275 3170 3275
@@
 Text GLabel 3245 3175 2    50   Input ~ 0
 BUZZER
-NoConn ~ 3170 3575
 $Comp
 L Device:D_Small D?
@@
 	1    0    0    -1
 $EndComp
+Text GLabel 3245 3575 2    50   Input ~ 0
+EN_VSW
+Wire Wire Line
+	3245 3575 3170 3575
+Text GLabel 3245 2075 2    50   Input ~ 0
+EN_24V
+Wire Wire Line
+	3245 2075 3170 2075
+Text GLabel 3245 1675 2    50   Input ~ 0
+EN_3.3V
+$Comp
+L Connector_Generic:Conn_01x04 J?
+U 1 1 62778B95
+P 3640 5630
+AR Path="/627661BA/62778B95" Ref="J?"  Part="1"
+AR Path="/62778B95" Ref="J5"  Part="1"
+F 0 "J5" H 3655 5880 50  0000 C CNN
+F 1 "Nozzle2 Board (Future)" H 3605 5290 50  0000 C CNN
+F 2 "Connector_PinHeader_2.54mm:PinHeader_1x04_P2.54mm_Vertical" H 3640 5630 50  0001 C CNN
+F 3 "~" H 3640 5630 50  0001 C CNN
+	1    3640 5630
+	-1   0    0    1
+$EndComp
+Text Notes 3275 5465 0    50   ~ 0
+EN_VSW
+Text Notes 3275 5565 0    50   ~ 0
+EN_24V
+Text Notes 3270 5660 0    50   ~ 0
+EN_3.3V
+Text Notes 3270 5760 0    50   ~ 0
+GND
+Text GLabel 3920 5430 2    50   Input ~ 0
+EN_VSW
+Text GLabel 3920 5530 2    50   Input ~ 0
+EN_24V
+Text GLabel 3920 5630 2    50   Input ~ 0
+EN_3.3V
+Wire Wire Line
+	3840 5430 3920 5430
+Wire Wire Line
+	3840 5530 3920 5530
+Wire Wire Line
+	3840 5630 3920 5630
+Wire Wire Line
+	3840 5730 3875 5730
+Wire Wire Line
+	3875 5730 3875 5770
+$Comp
+L power:GND #PWR?
+U 1 1 627BD38A
+P 3875 5770
+AR Path="/6231FCB3/627BD38A" Ref="#PWR?"  Part="1"
+AR Path="/627BD38A" Ref="#PWR0101"  Part="1"
+F 0 "#PWR0101" H 3875 5520 50  0001 C CNN
+F 1 "GND" H 3995 5665 50  0000 C CNN
+F 2 "" H 3875 5770 50  0001 C CNN
+F 3 "" H 3875 5770 50  0001 C CNN
+	1    3875 5770
+	1    0    0    -1
+$EndComp

Commit message: Updating Controller and Driver boards to version 0.6
Parts:
- removed J3: 2 x 10 Pinheader, Connector_PinSocket_2.54mm:PinSocket_2x10_P2.54mm_Vertical, symbol Connector_Generic:Conn_02x10_Odd_Even
- removed J5: Nozzle2 Board (Future), Connector_PinHeader_2.54mm:PinHeader_1x04_P2.54mm_Vertical, symbol Connector_Generic:Conn_01x04
- added J2: Plug, Connector_Hirose:Hirose_DF13C_CL535-0403-5-51_1x03-1MP_P1.25mm_Vertical, symbol Connector:Conn_01x03_Male
- added J3: Header, Connector_PinHeader_2.54mm:PinHeader_1x03_P2.54mm_Vertical, symbol Connector:Conn_01x03_Male
- added J5: Conn_02x12_Odd_Even, Connector_PinHeader_2.54mm:PinHeader_2x12_P2.54mm_Vertical, symbol Connector_Generic:Conn_02x12_Odd_Even
- added TP1: TestPoint, TestPoint:TestPoint_THTPad_1.5x1.5mm_Drill0.7mm, symbol Connector:TestPoint
- renumbered J2 to J4
Connections:
- net EN_VSW is gone; now on net USER1: U1.9 (IO33)
- net +3.3VDAC: now also J5.13 (Pin_13), J5.9 (Pin_9)
- net +3V3: now also J2.3 (Pin_3), J3.3 (Pin_3)
- net GND: now also J2.1 (Pin_1), J3.1 (Pin_1), J5.1 (Pin_1), J5.11 (Pin_11), J5.15 (Pin_15), J5.17 (Pin_17), J5.19 (Pin_19), J5.21 (Pin_21), J5.23 (Pin_23), J5.3 (Pin_3), J5.5 (Pin_5), J5.7 (Pin_7)
- net PH0: now also J5.2 (Pin_2)
- net PH1: now also J5.4 (Pin_4)
- net PH2: now also J5.6 (Pin_6)
- net PH3: now also J5.8 (Pin_8)
- net PH4: now also J5.10 (Pin_10)
- net PH5: now also J5.12 (Pin_12)
- net PH6: now also J5.14 (Pin_14)
- net PH7: now also J5.16 (Pin_16)
- net USER1: no longer U1.11 (IO26)
- net MOSI: now reaches U1.23 (IO15)
- net MOSI: now also J5.22 (Pin_22)
- net CS: now reaches U1.29 (IO5)
- net CS: now also J5.24 (Pin_24)
- net at U1.6 (IO34): now also TP1.1
- net EN_24V renamed SCLK
- net SCLK: now also J5.18 (Pin_18)
- net EN_3.3V renamed MISO
- net MISO: now also J5.20 (Pin_20)
- new net DAC2: J2.2 (Pin_2), J3.2 (Pin_2), U1.11 (IO26)
- no-connect marks 10 -> 7
Other:
- note added: "DAC2 or Spare GPIO Output"
- note removed: "1 easy to use spare RO GPIO"
- note removed: "2 extra spare strapping pin GPIO"
- note removed: "EN_24V"
- note removed: "EN_3.3V"
- note removed: "EN_VSW"
- note removed: "GND"

Commit message: Adding in version 0.7 KiACD design files
Parts:
- added H6: MH-M2, MountingHole:MountingHole_2.2mm_M2, symbol Mechanical:MountingHole
- C4: value 10uF -> 100nF
Other:
- moved on the sheet: H5
Changed lines of the file:
@@
 Sheet 1 2
 Title "Open-PyroJet Controller"
-Date "2022-05-09"
-Rev "0.6a"
+Date "2022-06-14"
+Rev "0.7"
 Comp "OPJ"
 Comment1 "PRL"
@@
 AR Path="/62340863" Ref="C4"  Part="1"
 F 0 "C4" H 1745 2000 50  0000 L CNN
-F 1 "10uF" H 1695 2165 50  0000 L CNN
+F 1 "100nF" H 1695 2165 50  0000 L CNN
 F 2 "Capacitor_SMD:C_0603_1608Metric" H 1665 2080 50  0001 C CNN
 F 3 "~" H 1665 2080 50  0001 C CNN
@@
 L Mechanical:MountingHole H?
 U 1 1 62CE5555
-P 7570 5680
+P 7560 5590
 AR Path="/6231FCB3/62CE5555" Ref="H?"  Part="1"
 AR Path="/62CE5555" Ref="H5"  Part="1"
-F 0 "H5" H 7670 5726 50  0000 L CNN
-F 1 "MH-M3" H 7670 5635 50  0000 L CNN
-F 2 "MountingHole:MountingHole_3.2mm_M3" H 7570 5680 50  0001 C CNN
-F 3 "~" H 7570 5680 50  0001 C CNN
-	1    7570 5680
+F 0 "H5" H 7660 5636 50  0000 L CNN
+F 1 "MH-M3" H 7660 5545 50  0000 L CNN
+F 2 "MountingHole:MountingHole_3.2mm_M3" H 7560 5590 50  0001 C CNN
+F 3 "~" H 7560 5590 50  0001 C CNN
+	1    7560 5590
 	1    0    0    -1
 $EndComp
@@
 Wire Wire Line
 	3245 3275 3170 3275
+$Comp
+L Mechanical:MountingHole H?
+U 1 1 62AC310F
+P 7560 5760
+AR Path="/6231FCB3/62AC310F" Ref="H?"  Part="1"
+AR Path="/62AC310F" Ref="H6"  Part="1"
+F 0 "H6" H 7660 5806 50  0000 L CNN
+F 1 "MH-M2" H 7660 5715 50  0000 L CNN
+F 2 "MountingHole:MountingHole_2.2mm_M2" H 7560 5760 50  0001 C CNN
+F 3 "~" H 7560 5760 50  0001 C CNN
+	1    7560 5760
+	1    0    0    -1
+$EndComp
 $EndSCHEMATC
