File: Printhead-Controller/UART.sch (KiCad schematic (older format))
At the start: 17 parts, among them J4 USB_B_Micro, U2 CP2102N-A01-GQFN28, U3 DMMT3904W

Commit message: Updating Controller and Driver boards to version 0.6
Parts:
- removed JP1, JP2: Jumper_NC_Small, Resistor_SMD:R_0402_1005Metric, symbol Device:Jumper_NC_Small
- R13, R14: footprint Resistor_SMD:R_0402_1005Metric -> Resistor_SMD:R_0603_1608Metric
- R15, R17: value 12K -> 10K; footprint Resistor_SMD:R_0402_1005Metric -> Resistor_SMD:R_0603_1608Metric
- renumbered J4 to J6
Connections:
- net Rx: now also U2.25 (RXD)
- net Tx: now also U2.26 (TXD)
- net EN renamed RESET
- net IO0 renamed BOOT
Other:
- note removed: "isolation jumpers"
Changed lines of the file:
@@
 encoding utf-8
 Sheet 2 2
-Title "Open-PyroJet-UART"
-Date "2022-03-22"
-Rev "0.5c2"
+Title "Open-PyroJet Controller - UART"
+Date "2022-05-09"
+Rev "0.6a"
 Comp "OPJ"
 Comment1 "PRL"
@@
 	5190 3990 5585 3990
 $Comp
-L power:GND #PWR035
+L power:GND #PWR037
 U 1 1 5EE7E8E5
 P 4170 4690
-F 0 "#PWR035" H 4170 4440 50  0001 C CNN
+F 0 "#PWR037" H 4170 4440 50  0001 C CNN
 F 1 "GND" H 4175 4517 50  0000 C CNN
 F 2 "" H 4170 4690 50  0001 C CNN
@@
 $EndComp
 NoConn ~ 5585 3590
-Text GLabel 7070 3690 2    50   Input ~ 0
+Text GLabel 6870 3690 2    50   Input ~ 0
 Tx
-Text GLabel 7065 3590 2    50   Input ~ 0
+Text GLabel 6865 3590 2    50   Input ~ 0
 Rx
-Wire Wire Line
-	6585 3590 6785 3590
 NoConn ~ 6585 5390
 NoConn ~ 6585 5290
@@
 NoConn ~ 6585 4690
 $Comp
-L power:GND #PWR036
+L power:GND #PWR038
 U 1 1 5EE816CF
 P 6085 5845
-F 0 "#PWR036" H 6085 5595 50  0001 C CNN
+F 0 "#PWR038" H 6085 5595 50  0001 C CNN
 F 1 "GND" H 6090 5672 50  0000 C CNN
 F 2 "" H 6085 5845 50  0001 C CNN
@@
 	6085 5790 6085 5820
 $Comp
-L power:+3V3 #PWR031
+L power:+3V3 #PWR033
 U 1 1 5EE82456
 P 6085 3035
-F 0 "#PWR031" H 6085 2885 50  0001 C CNN
+F 0 "#PWR033" H 6085 2885 50  0001 C CNN
 F 1 "+3V3" H 6100 3208 50  0000 C CNN
 F 2 "" H 6085 3035 50  0001 C CNN
@@
 	5985 2925 5985 3120
 $Comp
-L power:GND #PWR032
+L power:GND #PWR034
 U 1 1 5EE84AA7
 P 5460 3175
-F 0 "#PWR032" H 5460 2925 50  0001 C CNN
+F 0 "#PWR034" H 5460 2925 50  0001 C CNN
 F 1 "GND" H 5465 3002 50  0000 C CNN
 F 2 "" H 5460 3175 50  0001 C CNN
@@
 P 8175 4240
 F 0 "R15" V 7979 4240 50  0000 C CNN
-F 1 "12K" V 8070 4240 50  0000 C CNN
-F 2 "Resistor_SMD:R_0402_1005Metric" H 8175 4240 50  0001 C CNN
+F 1 "10K" V 8070 4240 50  0000 C CNN
+F 2 "Resistor_SMD:R_0603_1608Metric" H 8175 4240 50  0001 C CNN
 F 3 "~" H 8175 4240 50  0001 C CNN
 	1    8175 4240
@@
 P 8200 4810
 F 0 "R17" V 8004 4810 50  0000 C CNN
-F 1 "12K" V 8095 4810 50  0000 C CNN
-F 2 "Resistor_SMD:R_0402_1005Metric" H 8200 4810 50  0001 C CNN
+F 1 "10K" V 8095 4810 50  0000 C CNN
+F 2 "Resistor_SMD:R_0603_1608Metric" H 8200 4810 50  0001 C CNN
 F 3 "~" H 8200 4810 50  0001 C CNN
 	1    8200 4810
@@
 	8675 4420 8985 4420
 Text GLabel 7390 4620 0    50   Input ~ 0
-EN
+RESET
 Text GLabel 8985 4420 2    50   Input ~ 0
-IO0
+BOOT
 Text GLabel 8930 4620 2    50   Input ~ 0
 RTS
@@
 F 0 "R14" V 4809 3790 50  0000 C CNN
 F 1 "24K" V 4900 3790 50  0000 C CNN
-F 2 "Resistor_SMD:R_0402_1005Metric" H 5005 3790 50  0001 C CNN
+F 2 "Resistor_SMD:R_0603_1608Metric" H 5005 3790 50  0001 C CNN
 F 3 "~" H 5005 3790 50  0001 C CNN
 	1    5005 3790
@@
 U 1 1 5EA61456
 P 5330 3620
-F 0 "R13" V 5134 3620 50  0000 C CNN
-F 1 "47K" V 5225 3620 50  0000 C CNN
-F 2 "Resistor_SMD:R_0402_1005Metric" H 5330 3620 50  0001 C CNN
+F 0 "R13" H 5200 3550 50  0000 C CNN
+F 1 "47K" H 5200 3680 50  0000 C CNN
+F 2 "Resistor_SMD:R_0603_1608Metric" H 5330 3620 50  0001 C CNN
 F 3 "~" H 5330 3620 50  0001 C CNN
 	1    5330 3620
@@
 NoConn ~ 6585 4290
 $Comp
-L power:VBUS #PWR033
+L power:VBUS #PWR035
 U 1 1 60217A10
 P 4830 3565
-F 0 "#PWR033" H 4830 3415 50  0001 C CNN
+F 0 "#PWR035" H 4830 3415 50  0001 C CNN
 F 1 "VBUS" H 4845 3738 50  0000 C CNN
 F 2 "" H 4830 3565 50  0001 C CNN
@@
 Wire Wire Line
 	4830 3790 4830 3565
-Wire Wire Line
-	6585 3690 6785 3690
-$Comp
-L Device:Jumper_NC_Small JP2
-U 1 1 60033C77
-P 6885 3690
-F 0 "JP2" H 6995 3750 50  0000 C CNN
-F 1 "Jumper_NC_Small" H 6885 3811 50  0001 C CNN
-F 2 "Resistor_SMD:R_0402_1005Metric" H 6885 3690 50  0001 C CNN
-F 3 "~" H 6885 3690 50  0001 C CNN
-	1    6885 3690
-	1    0    0    -1
-$EndComp
-Wire Wire Line
-	6985 3690 7070 3690
-$Comp
-L Device:Jumper_NC_Small JP1
-U 1 1 600346D6
-P 6885 3590
-F 0 "JP1" H 7000 3650 50  0000 C CNN
-F 1 "Jumper_NC_Small" H 6885 3711 50  0001 C CNN
-F 2 "Resistor_SMD:R_0402_1005Metric" H 6885 3590 50  0001 C CNN
-F 3 "~" H 6885 3590 50  0001 C CNN
-	1    6885 3590
-	1    0    0    -1
-$EndComp
-Wire Wire Line
-	6985 3590 7065 3590
-Text Notes 6730 3805 0    50   ~ 0
-isolation jumpers
-$Comp
-L Connector:USB_B_Micro J4
+$Comp
+L Connector:USB_B_Micro J6
 U 1 1 5F9DBEB4
 P 4270 3990
-F 0 "J4" H 4327 4457 50  0000 C CNN
+F 0 "J6" H 4327 4457 50  0000 C CNN
 F 1 "USB_B_Micro" H 4327 4366 50  0000 C CNN
 F 2 "Pauls_KiCAD_Libraries:USB_Micro-B_C319160" H 4420 3940 50  0001 C CNN
@@
 	6085 5820 6085 5845
 $Comp
-L power:VBUS #PWR034
+L power:VBUS #PWR036
 U 1 1 5FDC33C9
 P 5040 4615
-F 0 "#PWR034" H 5040 4465 50  0001 C CNN
+F 0 "#PWR036" H 5040 4465 50  0001 C CNN
 F 1 "VBUS" H 5055 4788 50  0000 C CNN
 F 2 "" H 5040 4615 50  0001 C CNN
@@
 Wire Wire Line
 	7615 4240 8075 4240
+Wire Wire Line
+	6585 3590 6865 3590
+Wire Wire Line
+	6585 3690 6870 3690
 $EndSCHEMATC
